File: ruler_kicad.kicad_pcb (KiCad board)
At the start: 2 copper layers, 304.9 x 35 mm, 18 parts, among them U1 2EDL23N06PJXUMA1, U2 iC-HTG, U3 74LVC1G11

Commit message: Added the "M" after resistor sezes number (some of them didnt have them coz i forgot and not noticet))
Other:
- board text added: "0612_1632M"
- board text added: "0805_2012M"
- board text removed: "0612_1632"
- board text removed: "0805_2012"
- board text removed: "0815_2038"
Changed lines of the file:
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@@
 		)
 	)
-	(gr_text "0612_1632"
+	(gr_text "0612_1632M"
 		(at 94.4 140.1718 0)
 		(layer "F.SilkS")
@@
 		)
 	)
-	(gr_text "0805_2012"
+	(gr_text "0805_2012M\n"
 		(at 94.4 144.5968 0)
 		(layer "F.SilkS")
@@
 		)
 	)
-	(gr_text "0815_2038"
+	(gr_text "0815_2038M"
 		(at 118 132.395 0)
 		(layer "F.SilkS")
